Commit message: fix launch files

File: urdf/base_v0/base_mod.urdf.xacro (robot description, xacro)
@@ -259,6 +259,6 @@
     <joint name="${name}_footprint_joint" type="fixed">
       <origin xyz="0 0 0.051" rpy="0 0 0" />
-      <parent link="${name}_box_link"/>
-	  <child link="${name}_footprint" />
+      <parent link="${name}_footprint"/>
+      <child link="${name}_link" />
     </joint>
     <!-- visualize bellow -->
@@ -290,5 +290,5 @@
     </joint>
     <!-- base laser -->
-    <xacro:hokuyo_lx30_laser_v0 name="${name}_laser" parent="${name}_box" ros_topic="base_scan" update_rate="20" min_angle="-2.2689" max_angle="2.2689" >
+    <xacro:hokuyo_lx30_laser_v0 name="${name}_laser" parent="${name}" ros_topic="base_scan" update_rate="20" min_angle="-2.2689" max_angle="2.2689" >
       <origin xyz="${base_laser_x} ${base_laser_y} ${base_laser_z}" rpy="0 0 0" />
     </xacro:hokuyo_lx30_laser_v0>

File: urdf/pr2_mod.urdf.xacro (robot description, xacro)
@@ -157,5 +157,5 @@
       <updatePeriod>0.5</updatePeriod>
       <!-- TODO: maybe should rather be in world or map frame -->
-      <publishFrameId>base_link</publishFrameId>
+      <publishFrameId>base_footprint</publishFrameId>
     </plugin>
   </gazebo>

Commit message: spawn robot at 20,20, remove base_footprint collision to be sure

File: urdf/base_v0/base_mod.urdf.xacro (robot description, xacro)
@@ -248,12 +248,12 @@
         <material name="White" />
       </visual>
-      <collision>
-        <!-- represent base collision with a simple rectangular model, positioned by base_size_z s.t. top
-             surface of the collision box matches the top surface of the PR2 base -->
-        <origin xyz="0 0 ${0.051+base_collision_size_z/2}" rpy="0 0 0" />
-        <geometry>
-          <box size="0.001 0.001 0.001" />
-        </geometry>
-      </collision>
+<!--      <collision>-->
+<!--        &lt;!&ndash; represent base collision with a simple rectangular model, positioned by base_size_z s.t. top-->
+<!--             surface of the collision box matches the top surface of the PR2 base &ndash;&gt;-->
+<!--        <origin xyz="0 0 ${0.051+base_collision_size_z/2}" rpy="0 0 0" />-->
+<!--        <geometry>-->
+<!--          <box size="0.001 0.001 0.001" />-->
+<!--        </geometry>-->
+<!--      </collision>-->
     </link>
     <joint name="${name}_footprint_joint" type="fixed">
@@ -290,4 +290,5 @@
     </joint>
     <!-- base laser -->
+    <!-- NOTE: THIS SEEMS TO SLIP OFF OF base_link. I THINK IT WOULD HAVE TO BE ATTACHED TO base_box_link, BUT SEEMS IMPOSSIBLE TO CHANGE OR REMOVE WITHOUT CRASHING GAZEBO-->
     <xacro:hokuyo_lx30_laser_v0 name="${name}_laser" parent="${name}" ros_topic="base_scan" update_rate="20" min_angle="-2.2689" max_angle="2.2689" >
       <origin xyz="${base_laser_x} ${base_laser_y} ${base_laser_z}" rpy="0 0 0" />

Commit message: prevent robot tipping over: add damping, rm left arm initial joint position in gazebo

File: urdf/base_v0/base_mod.urdf.xacro (robot description, xacro)
@@ -159,5 +159,6 @@
 	  <limit effort="1000.0" lower="-100.0" upper="100.0" velocity="0.5"/>
 	  <axis xyz="1 0 0"/>
-	</joint>
+        <dynamics damping="1.0" friction="0.0" />
+    </joint>
 	<link name="${name}_y_link">
 	  <inertial>
@@ -181,5 +182,6 @@
 	  <axis xyz="0 1 0"/>
 	  <limit effort="1000.0" lower="-100.0" upper="100.0" velocity="0.5"/>
-	</joint>
+        <dynamics damping="1.0" friction="0.0" />
+    </joint>
 	<link name="${name}_theta_link">
 	  <inertial>
@@ -203,5 +205,6 @@
 	  <child link="${name}_theta_link"/>
 	  <axis xyz="0 0 1"/>
-	</joint>
+        <dynamics damping="1.0" friction="0.0" />
+    </joint>
     <!-- base_footprint is a fictitious link(frame) that is on the ground right below base_link origin,
          navigation stack dedpends on this frame -->
@@ -231,5 +234,6 @@
 	  <parent link="${name}_theta_link"/>
 	  <child link="${name}_box_link"/>
-	</joint>
+        <dynamics damping="1.0" friction="0.0" />
+    </joint>
     <!-- base_footprint is a fictitious link(frame) that is on the ground right below base_link origin,
          navigation stack dedpends on this frame -->

Commit message: more damping and friction to ensure robot does not fall over

File: urdf/base_v0/base_mod.urdf.xacro (robot description, xacro)
@@ -159,5 +159,5 @@
 	  <limit effort="1000.0" lower="-100.0" upper="100.0" velocity="0.5"/>
 	  <axis xyz="1 0 0"/>
-        <dynamics damping="1.0" friction="0.0" />
+        <dynamics damping="10.0" friction="0.1" />
     </joint>
 	<link name="${name}_y_link">
@@ -182,5 +182,5 @@
 	  <axis xyz="0 1 0"/>
 	  <limit effort="1000.0" lower="-100.0" upper="100.0" velocity="0.5"/>
-        <dynamics damping="1.0" friction="0.0" />
+        <dynamics damping="10.0" friction="0.1" />
     </joint>
 	<link name="${name}_theta_link">
@@ -205,5 +205,5 @@
 	  <child link="${name}_theta_link"/>
 	  <axis xyz="0 0 1"/>
-        <dynamics damping="1.0" friction="0.0" />
+        <dynamics damping="10.0" friction="0.1" />
     </joint>
     <!-- base_footprint is a fictitious link(frame) that is on the ground right below base_link origin,
@@ -234,5 +234,5 @@
 	  <parent link="${name}_theta_link"/>
 	  <child link="${name}_box_link"/>
-        <dynamics damping="1.0" friction="0.0" />
+        <dynamics damping="10.0" friction="0.1" />
     </joint>
     <!-- base_footprint is a fictitious link(frame) that is on the ground right below base_link origin,
